File: rudeboard.kicad_pcb (KiCad board)
At the start: 2 copper layers, 295.8 x 124.2 mm, 132 parts, among them U1 Elite-C

Commit message: fix silkscreen
- move dimensions to Dwgs.User
- move diodes
- reroute diodes
- remove unneeded silkscreen/artwork
Parts:
- removed G***: LOGO, Keebio_Parts:SquirtleSquadLeader
- moved D13 1.27 mm to (320.8, 74.4)
- moved D26 1.27 mm to (320.8, 93.5)
- moved D19 1.27 mm to (149.4, 93.5)
- moved D21 1.27 mm to (206.5, 93.5)
- moved D32 1.27 mm to (149.4, 112.5)
- moved D34 1.27 mm to (206.5, 112.5)
- moved D4 1.27 mm to (149.4, 74.4)
- moved D45 1.27 mm to (149.4, 131.6)
- moved D56 1.27 mm to (139.8, 150.6)
- moved D6 1.27 mm to (187.5, 74.4)
- moved D63 1.27 mm to (130.4, 169.7)
- moved D64 1.27 mm to (225.8, 169.5)
- moved D7 1.27 mm to (206.5, 74.4)
- moved D9 1.27 mm to (244.6, 74.4)
- moved D1 1.27 mm to (92.2, 74.4)
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Routing:
- net /row2: track 273.5 -> 276.1 mm
- net /col8: track 98.4 -> 96.9 mm
- net Net-(D26-Pad2): track 6.04 -> 7.31 mm
- net Net-(D13-Pad2): track 6.04 -> 7.31 mm
- net Net-(D9-Pad2): track 6.04 -> 7.31 mm
- net Net-(D7-Pad2): track 6.04 -> 7.31 mm
- net Net-(D64-Pad2): track 6.24 -> 7.51 mm
- net Net-(D63-Pad2): track 6.17 -> 7.44 mm
- net Net-(D6-Pad2): track 6.04 -> 7.31 mm
- net Net-(D56-Pad2): track 6.04 -> 7.31 mm
- net Net-(D45-Pad2): track 6.04 -> 7.31 mm
- net Net-(D4-Pad2): track 6.04 -> 7.31 mm
- net Net-(D34-Pad2): track 6.04 -> 7.31 mm
- net Net-(D32-Pad2): track 6.04 -> 7.31 mm
- net Net-(D21-Pad2): track 6.04 -> 7.31 mm
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Other:
- board text removed: "hangry#9198"
- board text removed: "rudeboard"
- board text removed: "rudeyboy#0420"
